File: LPmini-Prototype.brd (EAGLE design)
At the start: 50.8 x 25.3 mm, 46 parts, among them U1 ESD_TPD2E001, U2 SPX3819-3.3, U3 MCP73831T-2ACI/OT, X1 JSTPH, X2 16MHZ

Commit message: Add files via upload
Parts:
- removed D1: (no value), 0Joseph:0_JOSEPH_D0603
- added D2: MBR120, microbuilder:SOD-123
Connections:
- net VCC: now also D2.C; no longer D1.CA
- net VREF+: now also D2.A; no longer D1.AN
Routing:
- net VREF+: track 36.9 -> 40.6 mm
- net A2: track 7.79 -> 9.22 mm, vias 0 -> 1
- net A0: track 13.3 -> 12.0 mm
- net A1: track 10.5 -> 9.42 mm
- net VCC: track 97.2 -> 97.7 mm
- net GND: vias 43 -> 41
Changed lines of the file:
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@@
 <layer number="14" name="Route14" color="1" fill="6" visible="no" active="no"/>
 <layer number="15" name="Route15" color="4" fill="6" visible="no" active="no"/>
-<layer number="16" name="Bottom" color="1" fill="1" visible="no" active="yes"/>
+<layer number="16" name="Bottom" color="1" fill="1" visible="yes" active="yes"/>
 <layer number="17" name="Pads" color="2" fill="1" visible="yes" active="yes"/>
 <layer number="18" name="Vias" color="2" fill="1" visible="yes" active="yes"/>
@@
 <element name="U$5" library="0Joseph" package="SOLDER_JUMPER_3" value="3PT_SOLDER_JUMPER" x="36.83" y="3.683" rot="MR0"/>
 <element name="U$6" library="0Joseph" package="SOLDER_JUMPER_3" value="3PT_SOLDER_JUMPER" x="31.75" y="3.683" rot="MR0"/>
-<element name="D1" library="0Joseph" package="0_JOSEPH_D0603" value="" x="19.812" y="5.08" smashed="yes" rot="R180">
-<attribute name="NAME" x="20.447" y="4.445" size="0.8128" layer="34" ratio="16" rot="R180"/>
-<attribute name="VALUE" x="20.447" y="6.985" size="1.27" layer="27" rot="R180"/>
-</element>
 <element name="RST" library="0Joseph" package="PB_KMR2" value="PB_SMALL_SMD" x="9.906" y="4.191" smashed="yes" rot="R180">
 <attribute name="NAME" x="9.779" y="2.159" size="0.8128" layer="34" ratio="16" rot="R180" align="center"/>
@@
 <attribute name="NAME" x="15.367" y="2.159" size="0.8128" layer="34" ratio="16" rot="R180" align="center"/>
 </element>
+<element name="D2" library="microbuilder" package="SOD-123" value="MBR120" x="21.209" y="4.318"/>
 </elements>
 <signals>
@@
 <via x="25.146" y="18.161" extent="1-16" drill="0.3302"/>
 <via x="4.318" y="17.653" extent="1-16" drill="0.3302"/>
-<via x="24.13" y="2.794" extent="1-16" drill="0.3302"/>
 <contactref element="RST" pad="1B"/>
 <contactref element="RST" pad="1A"/>
@@
 <via x="1.778" y="5.461" extent="1-16" drill="0.3302"/>
 <via x="9.144" y="3.302" extent="1-16" drill="0.3302"/>
-<via x="21.971" y="5.588" extent="1-16" drill="0.3302"/>
 <via x="17.145" y="15.748" extent="1-16" drill="0.3302"/>
 <via x="13.843" y="14.859" extent="1-16" drill="0.3302"/>
@@
 <contactref element="JP1" pad="10"/>
 <contactref element="U$12" pad="79"/>
-<wire x1="24.925" y1="7.18" x2="24.071" y2="7.18" width="0.254" layer="1"/>
-<wire x1="24.071" y1="7.18" x2="23.876" y2="6.985" width="0.254" layer="1"/>
-<wire x1="23.876" y1="6.985" x2="23.876" y2="3.556" width="0.254" layer="1"/>
-<wire x1="23.876" y1="3.556" x2="21.59" y2="1.27" width="0.254" layer="1"/>
+<wire x1="21.59" y1="1.27" x2="22.098" y2="1.27" width="0.254" layer="16"/>
+<wire x1="22.098" y1="1.27" x2="26.162" y2="5.334" width="0.254" layer="16"/>
+<wire x1="26.162" y1="5.334" x2="26.162" y2="6.985" width="0.254" layer="16"/>
+<via x="26.162" y="6.985" extent="1-16" drill="0.3302"/>
+<wire x1="26.162" y1="6.985" x2="25.967" y2="7.18" width="0.254" layer="1"/>
+<wire x1="25.967" y1="7.18" x2="24.925" y2="7.18" width="0.254" layer="1"/>
 </signal>
 <signal name="A1">
@@
 <wire x1="24.925" y1="7.68" x2="23.936" y2="7.68" width="0.254" layer="1"/>
 <wire x1="23.936" y1="7.68" x2="23.368" y2="7.112" width="0.254" layer="1"/>
-<wire x1="23.368" y1="7.112" x2="23.368" y2="3.683" width="0.254" layer="1"/>
-<wire x1="23.368" y1="3.683" x2="22.098" y2="2.413" width="0.254" layer="1"/>
-<wire x1="22.098" y1="2.413" x2="20.193" y2="2.413" width="0.254" layer="1"/>
-<wire x1="20.193" y1="2.413" x2="19.05" y2="1.27" width="0.254" layer="1"/>
+<wire x1="21.59" y1="3.81" x2="19.05" y2="1.27" width="0.254" layer="1"/>
+<wire x1="23.368" y1="7.112" x2="23.368" y2="6.477" width="0.254" layer="1"/>
+<wire x1="23.368" y1="6.477" x2="21.59" y2="4.699" width="0.254" layer="1"/>
+<wire x1="21.59" y1="4.699" x2="21.59" y2="3.81" width="0.254" layer="1"/>
 </signal>
 <signal name="5">
@@
 <wire x1="24.925" y1="8.18" x2="23.801" y2="8.18" width="0.254" layer="1"/>
 <wire x1="23.801" y1="8.18" x2="22.86" y2="7.239" width="0.254" layer="1"/>
-<wire x1="21.971" y1="2.921" x2="22.86" y2="3.81" width="0.254" layer="1"/>
-<wire x1="22.86" y1="3.81" x2="22.86" y2="7.239" width="0.254" layer="1"/>
 <wire x1="16.51" y1="1.27" x2="17.272" y2="1.27" width="0.254" layer="1"/>
-<wire x1="17.272" y1="1.27" x2="18.923" y2="2.921" width="0.254" layer="1"/>
-<wire x1="18.923" y1="2.921" x2="21.971" y2="2.921" width="0.254" layer="1"/>
+<wire x1="17.272" y1="1.27" x2="18.669" y2="2.667" width="0.254" layer="1"/>
+<wire x1="18.669" y1="2.667" x2="19.558" y2="2.667" width="0.254" layer="1"/>
+<wire x1="19.558" y1="2.667" x2="21.082" y2="4.191" width="0.254" layer="1"/>
+<wire x1="22.86" y1="7.239" x2="22.86" y2="6.604" width="0.254" layer="1"/>
+<wire x1="22.86" y1="6.604" x2="21.082" y2="4.826" width="0.254" layer="1"/>
+<wire x1="21.082" y1="4.826" x2="21.082" y2="4.191" width="0.254" layer="1"/>
 </signal>
 <signal name="9">
@@
 <wire x1="30.48" y1="0.762" x2="30.48" y2="3.175" width="0.254" layer="1"/>
 <wire x1="35.56" y1="3.063" x2="35.448" y2="3.175" width="0.254" layer="1"/>
-<contactref element="D1" pad="CA"/>
 <wire x1="48.895" y1="7.62" x2="48.895" y2="8.89" width="0.254" layer="1"/>
 <contactref element="BSL" pad="1B"/>
@@
 <wire x1="15.4813" y1="3.391" x2="17.544" y2="3.391" width="0.254" layer="1"/>
 <wire x1="18.542" y1="7.159" x2="18.542" y2="5.969" width="0.254" layer="1"/>
-<wire x1="18.542" y1="5.969" x2="18.912" y2="5.599" width="0.254" layer="1"/>
-<wire x1="18.912" y1="5.599" x2="18.912" y2="5.08" width="0.254" layer="1"/>
-<wire x1="18.912" y1="5.08" x2="18.912" y2="4.18" width="0.254" layer="1"/>
-<wire x1="18.912" y1="4.18" x2="18.123" y2="3.391" width="0.254" layer="1"/>
-<wire x1="18.123" y1="3.391" x2="17.544" y2="3.391" width="0.254" layer="1"/>
+<wire x1="18.432" y1="3.391" x2="17.544" y2="3.391" width="0.254" layer="1"/>
 <wire x1="15.4813" y1="3.391" x2="15.4813" y2="4.1783" width="0.254" layer="1"/>
 <wire x1="15.4813" y1="4.1783" x2="15.494" y2="4.191" width="0.254" layer="1"/>
@@
 <wire x1="43.18" y1="0.762" x2="43.18" y2="1.905" width="0.254" layer="1"/>
 <wire x1="43.18" y1="1.905" x2="48.895" y2="7.62" width="0.254" layer="1"/>
+<contactref element="D2" pad="C"/>
+<wire x1="18.432" y1="3.391" x2="19.359" y2="4.318" width="0.254" layer="1"/>
+<wire x1="18.542" y1="5.969" x2="19.359" y2="5.152" width="0.254" layer="1"/>
+<wire x1="19.359" y1="5.152" x2="19.359" y2="4.318" width="0.254" layer="1"/>
 </signal>
 <signal name="N$25">
@@
 <wire x1="24.638" y1="0" x2="12.7" y2="0" width="0.254" layer="1"/>
 <wire x1="12.7" y1="0" x2="11.43" y2="1.27" width="0.254" layer="1"/>
-<contactref element="D1" pad="AN"/>
 <wire x1="11.43" y1="1.27" x2="13.081" y2="2.921" width="0.254" layer="16"/>
-<wire x1="13.081" y1="2.921" x2="19.304" y2="2.921" width="0.254" layer="16"/>
-<wire x1="19.304" y1="2.921" x2="20.701" y2="4.318" width="0.254" layer="16"/>
-<via x="20.701" y="4.318" extent="1-16" drill="0.3048"/>
-<wire x1="20.701" y1="4.318" x2="20.701" y2="5.069" width="0.254" layer="1"/>
-<wire x1="20.701" y1="5.069" x2="20.712" y2="5.08" width="0.254" layer="1"/>
+<wire x1="13.081" y1="2.921" x2="22.733" y2="2.921" width="0.254" layer="16"/>
+<contactref element="D2" pad="A"/>
+<wire x1="22.733" y1="2.921" x2="24.13" y2="4.318" width="0.254" layer="16"/>
+<via x="24.13" y="4.318" extent="1-16" drill="0.3302"/>
+<wire x1="24.13" y1="4.318" x2="23.059" y2="4.318" width="0.254" layer="1"/>
 </signal>
 </signals>
