File: LPmini-Prototype.brd (EAGLE design)
At the start: 50.8 x 25.3 mm, 46 parts, among them U1 ESD_TPD2E001, U2 SPX3819-3.3, U3 MCP73831T-2ACI/OT, X1 JSTPH, X2 16MHZ

Commit message: Add files via upload
Parts:
- removed U$12: TI_MSP430_V16_INTERN_F552X---PN80, 0Joseph:TI_MSP430_V16_INTERN_PN80
- added JP2: PINHD_2X05SMD, 0Joseph:2X05-SMALL_SMD
- added U4: ESD_TPD2E001, 0Joseph:PROJECT7264_TPD2E001-DRL
- R8: value 10K\ -> 10K
- U$7: value PINHD_2X05SMD -> (none); device 0Joseph:2X05-SMALL_SMD -> 0Joseph:TITAN_LOGO
- U1: value ESD_TPD2E001 -> TI_MSP430_V16_INTERN_F552X---PN80; device 0Joseph:PROJECT7264_TPD2E001-DRL -> 0Joseph:TI_MSP430_V16_INTERN_PN80
- moved U$7 30.9 mm to (15.9, 11.6), flipped to the bottom, turned to 0 degrees
- moved U1 24.9 mm to (31.8, 11.4), turned to 90 degrees
Connections:
- removed net N$14: U$12.39
- net +5V: now also U1.65; no longer U$12.65
- net 10: now also U1.57; no longer U$12.57
- net 11: now also U1.58; no longer U$12.58
- net 12: now also U1.59; no longer U$12.59
- net 13: now also U1.60; no longer U$12.60
- net 5: now also U1.42; no longer U$12.42
- net 6: now also U1.55; no longer U$12.55
- net 9: now also U1.56; no longer U$12.56
- net A0: now also U1.77; no longer U$12.77
- net A0_RX: now also U1.41; no longer U$12.41
- net A0_TX: now also U1.40; no longer U$12.40
- net A1: now also U1.78; no longer U$12.78
- net A1_RX: now also U1.52; no longer U$12.52
- net A1_SCK: now also U1.45; no longer U$12.45
- net A1_TX: now also U1.51; no longer U$12.51
- net A2: now also U1.79; no longer U$12.79
- net A3: now also U1.80; no longer U$12.80
- net A4: now also U1.1; no longer U$12.1
- net A5: now also U1.2; no longer U$12.2
- net B0_SCL: now also U1.38; no longer U$12.38
- net B0_SDA: now also U1.37; no longer U$12.37
- net B1_SCK: now also U1.48; no longer U$12.48
- net B1_SCL: now also U1.47; no longer U$12.47
- net B1_SDA: now also U1.46; no longer U$12.46
- net D_N: now also U1.64, U4.2, U4.5; no longer U$12.64, U1.2, U1.5
- net D_P: now also U1.62, U4.3; no longer U$12.62, U1.3
- net GND: now also JP2.2, JP2.3, JP2.5, U1.14, U1.19, U1.49, U1.61, U1.68, U4.4; no longer U$12.14, U$12.19, U$12.49, U$12.61, U$12.68, U$7.2, U$7.3, U$7.5, U1.4
- net N$23: now also U1.66; no longer U$12.66
- net N$24: now also U1.67; no longer U$12.67
- net N$25: now also U1.20; no longer U$12.20
- net N$40: now also U1.69; no longer U$12.69
- net N$6: now also U1.63; no longer U$12.63
- net RST: now also JP2.6, U1.76; no longer U$12.76, U$7.6
- net TCK: now also JP2.9, U1.75; no longer U$12.75, U$7.9
- net TDI: now also JP2.7, U1.73; no longer U$12.73, U$7.7
- net TDO: now also JP2.8, U1.72; no longer U$12.72, U$7.8
- net TMS: now also JP2.10, U1.74; no longer U$12.74, U$7.10
- net VBUS: now also U4.1; no longer U1.1
- net VCC: now also JP2.1, U1.11, U1.18, U1.50; no longer U$12.11, U$12.18, U$12.50, U$7.1
- net VREF+: now also U1.9; no longer U$12.9
