File: LPmini-Prototype_1.2.brd (EAGLE design)
At the start: 50.8 x 22.9 mm, 48 parts, among them U1 TI_MSP430_V16_INTERN_F552X---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, U2 SPX3819-3.3, U3 MCP73831T-2ACI/OT, U4 ESD_TPD2E001, X1 JSTPH, X2 16MHZ

Commit message: Add files via upload
Changed lines of the file:
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@@
 <setting verticaltext="up"/>
 </settings>
-<grid distance="100" unitdist="mil" unit="mil" style="lines" multiple="1" display="yes" altdistance="0.025" altunitdist="inch" altunit="inch"/>
+<grid distance="5" unitdist="mil" unit="mil" style="lines" multiple="1" display="yes" altdistance="0.025" altunitdist="inch" altunit="inch"/>
 <layers>
 <layer number="1" name="Top" color="4" fill="1" visible="yes" active="yes"/>
@@
 <via x="8.001" y="16.129" extent="1-16" drill="0.3302"/>
 <via x="10.16" y="20.066" extent="1-16" drill="0.3302"/>
-<via x="10.541" y="12.954" extent="1-16" drill="0.3302"/>
+<via x="10.16" y="12.827" extent="1-16" drill="0.3302"/>
 <via x="33.02" y="0.635" extent="1-16" drill="0.3302"/>
 <via x="40.513" y="10.287" extent="1-16" drill="0.3302"/>
@@
 <contactref element="U3" pad="3"/>
 <contactref element="C3" pad="1"/>
-<wire x1="12.065" y1="16.002" x2="16.256" y2="16.002" width="0.254" layer="1"/>
+<wire x1="12.7" y1="16.002" x2="16.256" y2="16.002" width="0.254" layer="1"/>
 <wire x1="16.256" y1="16.002" x2="17.018" y2="16.764" width="0.254" layer="1"/>
 <wire x1="17.018" y1="16.764" x2="17.018" y2="17.526" width="0.254" layer="1"/>
@@
 <wire x1="16.51" y1="21.59" x2="16.51" y2="22.86" width="1.524" layer="16"/>
 <wire x1="16.51" y1="21.59" x2="16.51" y2="22.86" width="1.524" layer="1"/>
-<wire x1="12.065" y1="16.002" x2="11.667" y2="15.604" width="0.254" layer="1"/>
-<wire x1="11.667" y1="15.604" x2="11.16" y2="15.604" width="0.254" layer="1"/>
+<wire x1="12.7" y1="16.002" x2="12.302" y2="15.604" width="0.254" layer="1"/>
+<wire x1="12.302" y1="15.604" x2="11.16" y2="15.604" width="0.254" layer="1"/>
 </signal>
 <signal name="13">
@@
 <wire x1="6.35" y1="22.86" x2="6.35" y2="22.86" width="0" layer="19" extent="1-16"/>
 </signal>
-<signal name="N$10">
-<wire x1="-18.288" y1="19.431" x2="-2.54" y2="19.431" width="0" layer="19" extent="1-16"/>
-</signal>
 <signal name="N$11">
