File: LPmini-Prototype_1.2/LPmini-Prototype_1.2.brd (EAGLE design)
At the start: 50.8 x 22.9 mm, 48 parts, among them U1 TI_MSP430_V16_INTERN_F552X---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, U2 SPX3819-3.3, U3 MCP73831T-2ACI/OT, U4 ESD_TPD2E001, X1 JSTPH, X2 16MHZ

Commit message: Add files via upload
Connections:
- removed net +5V: C24.1, U1.65
- new net N$2: U$11.1
- new net N$7: U$11.2
- new net N$8: U$11.3
- new net N$9: U$11.4
- net VBUS: now also C24.1, U1.65
Routing:
- net N$2: track 10.2 -> 2.54 mm, vias 0 -> 1
- net VBUS: track 39.3 -> 44.6 mm, vias 3 -> 4
- net +5V: track 3.61 -> 0.00 mm
- net N$9: track 0.00 -> 2.54 mm, vias 0 -> 1
- net N$8: track 0.00 -> 2.54 mm, vias 0 -> 1
- net N$7: track 0.00 -> 2.54 mm, vias 0 -> 1
- net VREF+: vias 2 -> 3
- net VCC: vias 5 -> 6
- net VBAT: vias 1 -> 2
- net TCB: vias 0 -> 1
- net TCA: vias 0 -> 1
- net SCK: vias 0 -> 1
- net RST_BTN: vias 2 -> 3
- net RDB: vias 0 -> 1
- net RDA: vias 0 -> 1
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