File: LPmini-Prototype_1.2/LPmini-Prototype_1.2.sch (EAGLE design)
At the start: 47 parts, among them U1 TI_MSP430_V16_INTERN_F552X---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, U2 SPX3819-3.3, U3 MCP73831T-2ACI/OT, U4 ESD_TPD2E001, X1 JSTPH, X2 16MHZ

Commit message: Add files via upload
Connections:
- removed net +5V: C24.1, U1.65
- new net N$2: U$11.1
- new net N$7: U$11.2
- new net N$8: U$11.3
- new net N$9: U$11.4
- net VBUS: now also C24.1, U1.65
Other:
- note removed: "BREAKOUTS"
